File: KiCAD_simulations/Full_Bridge/Full_Bridge/Full_Bridge.kicad_sch (KiCad schematic)
At the start: 7 parts

Commit message: updates
Parts:
- removed C1: 100uF, symbol pspice:C
- added D5, D99: 1N4001, Diode_THT:D_DO-41_SOD81_P10.16mm_Horizontal, symbol Diode:1N4001
- added R2, R3: 10k, symbol pspice:R
- added R4: 10K, symbol pspice:R
- added V2: sin(0 50 50), symbol pspice:VSOURCE
- D1, D2, D3: Spice_Node_Sequence (none) -> 2 1
- R1: value 10K -> 10k
- V1: value dc 0 ac 220 -> sin(0 50 50); Spice_Model dc 0 ac 20 sin(0 220 50 0) -> (none); Spice_Netlist_Enabled Y -> (none); Spice_Primitive V -> (none)
Connections:
- net 0: now also D3.1 (K), R1.2, V1.2 (E2), D5.2 (A), R3.2, V2.2 (E2); no longer D2.1 (K), D4.1 (K), R1.1
- net Vin: now also D4.2 (A); no longer D2.2 (A)
- removed net Vother: D3.1 (K), D4.2 (A), V1.2 (E2)
- net vout renamed Vout2
- net Vout2: now also R2.2; no longer R1.2
- new net: D2.1 (K), D99.2 (A), V2.1 (E1)
- new net Vout: D4.1 (K), D5.1 (K), R2.1
- new net bitch: D99.1 (K), R4.1
- new net bitch2: D2.2 (A), R1.1
- new net post: R3.1, R4.2
Other:
- note added: ".tran 1m 50m"
- note removed: ".tran .5u 200m"

Commit message: updates
Parts:
- added C1: 10uF, symbol pspice:C
Connections:
- net Vout: now also C1.1
- net Vout2: now also C1.2
Changed lines of the file:
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@@
   (junction (at 171.45 78.74) (diameter 0) (color 0 0 0 0)
   )
+  (junction (at 200.66 83.82) (diameter 0) (color 0 0 0 0)
+  )
   (junction (at 181.61 83.82) (diameter 0) (color 0 0 0 0)
   )
@@
   (junction (at 74.93 63.5) (diameter 0) (color 0 0 0 0)
   )
+  (junction (at 200.66 96.52) (diameter 0) (color 0 0 0 0)
+  )
   (junction (at 158.75 86.36) (diameter 0) (color 0 0 0 0)
   )
@@
     (stroke (width 0) (type default) (color 0 0 0 0))
   )
+  (wire (pts (xy 200.66 83.82) (xy 212.09 83.82))
+    (stroke (width 0) (type default) (color 0 0 0 0))
+  )
   (wire (pts (xy 74.93 88.9) (xy 74.93 96.52))
     (stroke (width 0) (type default) (color 0 0 0 0))
   )
+  (wire (pts (xy 200.66 96.52) (xy 212.09 96.52))
+    (stroke (width 0) (type default) (color 0 0 0 0))
+  )
   (wire (pts (xy 170.18 91.44) (xy 173.99 91.44))
     (stroke (width 0) (type default) (color 0 0 0 0))
@@
     (stroke (width 0) (type default) (color 0 0 0 0))
   )
-  (wire (pts (xy 181.61 83.82) (xy 212.09 83.82))
+  (wire (pts (xy 181.61 83.82) (xy 200.66 83.82))
     (stroke (width 0) (type default) (color 0 0 0 0))
   )
@@
     (stroke (width 0) (type default) (color 0 0 0 0))
   )
-  (wire (pts (xy 156.21 96.52) (xy 212.09 96.52))
+  (wire (pts (xy 156.21 96.52) (xy 200.66 96.52))
     (stroke (width 0) (type default) (color 0 0 0 0))
   )
@@
     (pin "2")
   )
+  (symbol (lib_id "pspice:C") (at 200.66 90.17 0) (unit 1)
+    (in_bom yes) (on_board yes) (fields_autoplaced)
+    (property "Reference" "C1" (id 0) (at 205.74 88.8999 0)
+      (effects (font (size 1.27 1.27)) (justify left))
+    )
+    (property "Value" "10uF" (id 1) (at 205.74 91.4399 0)
+      (effects (font (size 1.27 1.27)) (justify left))
+    )
+    (property "Footprint" "" (id 2) (at 200.66 90.17 0)
+      (effects (font (size 1.27 1.27)) hide)
+    )
+    (property "Datasheet" "~" (id 3) (at 200.66 90.17 0)
+      (effects (font (size 1.27 1.27)) hide)
+    )
+    (pin "1")
+    (pin "2")
+  )
   (symbol (lib_id "pspice:R") (at 97.79 100.33 0) (unit 1)
     (in_bom yes) (on_board yes) (fields_autoplaced)
@@
       (effects (font (size 1.27 1.27)) hide)
     )
-    (property "Spice_Node_Sequence" "2 1" (id 8) (at 86.36 63.5 0)
+    (property "Spice_Node_Sequence" "2 1" (id 9) (at 86.36 63.5 0)
       (effects (font (size 1.27 1.27)) hide)
     )
@@
       (reference "#GND02") (unit 1) (value "0") (footprint "")
     )
+    (path "/1b02276b-42a3-440e-a040-898e1c5e6bfd"
+      (reference "C1") (unit 1) (value "10uF") (footprint "")
+    )
     (path "/5f8e6361-a069-4180-bf71-496a71abad2f"
